Commit message: updating vito_robot

File: robot/vito_soma.urdf.xacro (robot description, xacro)
@@ -34,9 +34,9 @@
   <!-- TORSO -->
   <xacro:model_torso name="torso" parent="vito_anchor">
-    <origin xyz="0 0 0"/>
+    <origin xyz="0 0 0.1" rpy="0 0 0"/>
   </xacro:model_torso>
   <!-- LEFT ARM -->
 <!--   <xacro:kuka_lwr name="left_arm" parent="vito_anchor">
-    <origin xyz="-0.165 -0.1085854 0.390" rpy="1.5707963267948966 0.5235987010713441 -0.5235990737060282"/>
+    <origin xyz="-0.1650   -0.0000    0.3814" rpy="-2.1588   -0.4478    1.8518"/>
   </xacro:kuka_lwr> -->
   <!-- LEFT SOFTHAND -->
@@ -47,5 +47,6 @@
   <!-- RIGHT ARM -->
   <xacro:kuka_lwr name="right_arm" parent="vito_anchor">
-    <origin xyz="-0.165 0.10858 0.390" rpy="-1.5707963267948966 -0.5235987010713441 0.5235990737060282"/>
+    <!-- <origin xyz="-0.165 0.10858 0.490" rpy="-1.5707963267948966 -0.5235987010713441 0.5235990737060282"/> -->
+    <origin xyz="-0.1650    0.0000    0.5986" rpy="-0.2810   -0.4478   0.5880"/>
   </xacro:kuka_lwr>
   <!-- RIGHT SOFTHAND -->
