Commit message: add modifies for param position box

File: urdf/cube.urdf.xacro (robot description, xacro)
@@ -11,5 +11,5 @@
 			<origin xyz="0 0 0" rpy="0 0 0"/>
 			<geometry>
-				<box size="0.06 0.06 0.06"/>
+				<box size="0.046 0.127 0.183"/>
 			</geometry>
 		</visual>
@@ -17,5 +17,5 @@
 			<origin xyz="0 0 0" rpy="0 0 0"/>
 			<geometry>
-				<box size="0.06 0.06 0.06"/>
+				<box size="0.046 0.127 0.183"/>
 			</geometry>
 		</collision>

Commit message: add test file

File: urdf/cube.urdf.xacro (robot description, xacro)
@@ -11,5 +11,5 @@
 			<origin xyz="0 0 0" rpy="0 0 0"/>
 			<geometry>
-				<box size="0.046 0.127 0.183"/>
+				<box size="0.063 0.063 0.188"/>
 			</geometry>
 		</visual>
@@ -17,5 +17,5 @@
 			<origin xyz="0 0 0" rpy="0 0 0"/>
 			<geometry>
-				<box size="0.046 0.127 0.183"/>
+				<box size="0.063 0.063 0.188"/>
 			</geometry>
 		</collision>

Commit message: add modif

File: urdf/cube.urdf.xacro (robot description, xacro)
@@ -11,5 +11,5 @@
 			<origin xyz="0 0 0" rpy="0 0 0"/>
 			<geometry>
-				<box size="0.063 0.063 0.188"/>
+				<box size="0.062 0.110 0.094"/>
 			</geometry>
 		</visual>
@@ -17,5 +17,5 @@
 			<origin xyz="0 0 0" rpy="0 0 0"/>
 			<geometry>
-				<box size="0.063 0.063 0.188"/>
+				<box size="0.062 0.110 0.094"/>
 			</geometry>
 		</collision>
